File: schematic.brd (EAGLE design)
At the start: 100 x 59.7 mm, 25 parts

Commit message: akjdf;sjf
Parts:
- removed U$1: BUCK-CONVERTER, buck-converter:BUCK-CONVERTER
- added PWR: (no value), pinhead:1X02
- added U$2: BUCK-CONVERTER, mine:BUCK-CONVERTER
- moved RED 91.4 mm to (3.81, 12.7), turned to 90 degrees
- moved YELLOW 91.4 mm to (3.81, 21.6), turned to 90 degrees
- moved GREEN 91.4 mm to (3.81, 30.5), turned to 90 degrees
- moved FAN2 85.7 mm to (90.8, 53.3), turned to 270 degrees
- moved IRL540N 84.0 mm to (90.2, 47.6)
- moved POWER_JACK 83.8 mm to (10.2, 61.0)
- moved R1 80.1 mm to (10.2, 7.62), turned to 270 degrees
- moved R4 78.4 mm to (90.2, 37.5)
- moved R2 77.1 mm to (10.2, 20.3), turned to 270 degrees
- moved R3 76.9 mm to (10.2, 33.0), turned to 270 degrees
- moved FAN1 68.1 mm to (85.1, 53.3), turned to 270 degrees
- moved SG90 48.9 mm to (33.0, 6.35)
- moved INCAP 44.6 mm to (21.6, 5.08), turned to 180 degrees
- moved ESP32 43.2 mm to (69.8, 17.8), turned to 0 degrees
- moved OUTCAP 31.4 mm to (34.3, 12.7), turned to 270 degrees
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Connections:
- net MS1_X renamed N$11
- net MS1_Y renamed N$5
- net MS2_X renamed N$12
- net MS2_Y renamed N$9
- net MS3_X renamed N$13
- net MS3_Y renamed N$10
- net N$32 renamed FAN_PW
- removed net N$15: DRIVER_X./EN, ESP32.11
- removed net N$19: DRIVER_Y./EN, ESP32.8
- removed net N$2: DRIVER_X.STEP, ESP32.12
- removed net N$23: ESP32.37, RED.A
- removed net N$25: GREEN.K, R1.1
- removed net N$26: ESP32.33, GREEN.A
- removed net N$27: ESP32.36, YELLOW.A
- removed net N$29: R3.1, RED.K
- removed net N$30: ESP32.7, SG90.1
- removed net N$31: ESP32.28, IRL540N.G, R4.1
- removed net N$4: DRIVER_Y.DIR, ESP32.10
- removed net N$5 (its old number): DRIVER_Y.STEP, ESP32.9
- new net FAN_EN: ESP32.25, IRL540N.G, R4.1
- new net GREEN_LED: ESP32.6, GREEN.A
- new net N$21: R1.1, RED.K
- new net N$8: GREEN.K, R3.1
- new net RED_LED: ESP32.8, RED.A
- new net SERVO: ESP32.5, SG90.1
- new net X_DIR: DRIVER_X.DIR, ESP32.31
- new net X_EN: DRIVER_X./EN, ESP32.29
- new net X_STEP: DRIVER_X.STEP, ESP32.30
- new net YELLOW_LED: ESP32.7, YELLOW.A
- new net Y_DIR: DRIVER_Y.DIR, ESP32.33
- new net Y_EN: DRIVER_Y./EN, ESP32.37
- new net Y_STEP: DRIVER_Y.STEP, ESP32.36
- net +12V: now also U$2.VIN1, U$2.VIN2; no longer U$1.VIN
- net +3V3: now also PWR.2; no longer ESP32.1
- net +5V: now also U$2.VOUT1, U$2.VOUT2; no longer U$1.VOUT
- net GND: now also U$2.GND@1, U$2.GND@2, U$2.GND@3, U$2.GND@4; no longer U$1.GND@1, U$1.GND@2
- net N$1: now also ESP32.1, PWR.1; no longer DRIVER_X.DIR, ESP32.13
Routing:
- net +12V: track 0.00 -> 146.3 mm
- net +3V3: track 0.00 -> 124.1 mm, vias 0 -> 5
- net GREEN_LED: track 0.00 -> 78.5 mm
- net YELLOW_LED: track 0.00 -> 74.3 mm
- net RED_LED: track 0.00 -> 67.3 mm
- net Y_EN: track 0.00 -> 42.5 mm
- net +5V: track 0.00 -> 42.1 mm
- net Y_DIR: track 0.00 -> 40.8 mm
- net Y_STEP: track 0.00 -> 32.7 mm
- net X_EN: track 0.00 -> 26.4 mm
- net SERVO: track 0.00 -> 25.7 mm
- net FAN_EN: track 0.00 -> 25.2 mm
- net GND: track 0.00 -> 24.7 mm
- net FAN_PW: track 0.00 -> 15.4 mm
- net N$1: track 0.00 -> 11.0 mm
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Other:
- board size 100 x 59.7 mm -> 99.7 x 58.4 mm
- board text added: "+"
- board text added: "-"
- board text added: "Servo"

Commit message: kasjf;lkdsjf
Parts:
- renumbered PWR to ESP_PWR
Connections:
- net N$1 renamed ESP_PWR
- net N$21 renamed RED_R1
- net N$7 renamed YELLOW_R2
- net N$8 renamed GREEN_R3
- net GREEN_LED: now also ESP32.8; no longer ESP32.6
- net RED_LED: now also ESP32.10; no longer ESP32.8
- net SERVO: now also ESP32.7; no longer ESP32.5
- net YELLOW_LED: now also ESP32.9; no longer ESP32.7
Routing:
- net GREEN_LED: track 78.5 -> 83.9 mm
- net SERVO: track 25.7 -> 30.9 mm
- net YELLOW_LED: track 74.3 -> 79.3 mm
- net RED_LED: track 67.3 -> 72.4 mm
- net +3V3: track 124.1 -> 127.4 mm
Changed lines of the file:
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@@
 <setting verticaltext="up"/>
 </settings>
-<grid distance="100" unitdist="mil" unit="mil" style="lines" multiple="1" display="yes" altdistance="5" altunitdist="mil" altunit="mil"/>
+<grid distance="5" unitdist="mil" unit="mil" style="lines" multiple="1" display="yes" altdistance="5" altunitdist="mil" altunit="mil"/>
 <layers>
 <layer number="1" name="Top" color="4" fill="1" visible="yes" active="yes"/>
@@
 </element>
 <element name="U$2" library="mine" package="BUCK-CONVERTER" value="BUCK-CONVERTER" x="30.48" y="25.4" smashed="yes" rot="R270"/>
-<element name="PWR" library="pinhead" library_urn="urn:adsk.eagle:library:325" package="1X02" package3d_urn="urn:adsk.eagle:package:22435/2" value="" x="38.1" y="12.7" smashed="yes" rot="R90">
-<attribute name="NAME" x="41.4782" y="10.5918" size="1.27" layer="25" ratio="10" rot="R90"/>
+<element name="ESP_PWR" library="pinhead" library_urn="urn:adsk.eagle:library:325" package="1X02" package3d_urn="urn:adsk.eagle:package:22435/2" value="" x="38.1" y="12.7" smashed="yes" rot="R90">
+<attribute name="NAME" x="41.3512" y="8.4328" size="1.27" layer="25" ratio="10" rot="R90"/>
 <attribute name="VALUE" x="41.275" y="10.16" size="1.27" layer="27" rot="R90"/>
 </element>
@@
 <wire x1="40.64" y1="20.828" x2="40.64" y2="24.765" width="0.762" layer="1"/>
 <wire x1="38.862" y1="19.05" x2="36.83" y2="19.05" width="0.762" layer="1"/>
-<wire x1="36.83" y1="16.51" x2="36.83" y2="19.05" width="0.762" layer="1"/>
-<wire x1="36.83" y1="16.51" x2="34.29" y2="13.97" width="0.762" layer="1"/>
+<wire x1="36.83" y1="15.24" x2="36.83" y2="19.05" width="0.762" layer="1"/>
 <wire x1="40.64" y1="34.798" x2="40.64" y2="36.195" width="0.762" layer="1"/>
 <wire x1="52.07" y1="35.56" x2="51.643196875" y2="35.0478375" width="0.762" layer="1"/>
@@
 <via x="69.596" y="34.29" extent="1-16" drill="0.35"/>
 <wire x1="69.596" y1="36.576" x2="69.596" y2="34.29" width="0.762" layer="1"/>
-<contactref element="PWR" pad="2"/>
-<wire x1="36.83" y1="16.51" x2="36.83" y2="15.24" width="0.762" layer="1"/>
+<contactref element="ESP_PWR" pad="2"/>
 <wire x1="36.83" y1="15.24" x2="38.1" y2="13.97" width="0.762" layer="1"/>
+<wire x1="34.29" y1="13.97" x2="35.56" y2="13.97" width="0.762" layer="1"/>
+<wire x1="35.56" y1="13.97" x2="36.957" y2="13.97" width="0.762" layer="1"/>
+<wire x1="36.957" y1="13.97" x2="38.1" y2="13.97" width="0.762" layer="1"/>
+<wire x1="36.83" y1="15.24" x2="36.83" y2="14.097" width="0.762" layer="1"/>
+<wire x1="36.83" y1="14.097" x2="36.957" y2="13.97" width="0.762" layer="1"/>
+<wire x1="36.83" y1="15.24" x2="35.56" y2="13.97" width="0.762" layer="1"/>
 </signal>
 <signal name="N$6">
@@
 <wire x1="27.94" y1="12.192" x2="26.67" y2="10.668" width="1.27" layer="1"/>
 </signal>
-<signal name="RED_LED">
-<contactref element="ESP32" pad="8"/>
-<wire x1="64.77" y1="6.35" x2="59.69" y2="1.27" width="0.508" layer="1"/>
-<contactref element="RED" pad="A"/>
-<wire x1="13.97" y1="1.27" x2="3.81" y2="11.43" width="0.508" layer="1"/>
-<wire x1="59.69" y1="1.27" x2="13.97" y2="1.27" width="0.508" layer="1"/>
-</signal>
 <signal name="FAN_PW">
 <contactref element="IRL540N" pad="D"/>
@@
 <wire x1="88.265" y1="52.07" x2="90.17" y2="50.165" width="1.016" layer="1"/>
 </signal>
-<signal name="N$7">
+<signal name="YELLOW_R2">
 <contactref element="R2" pad="1"/>
 <contactref element="YELLOW" pad="K"/>
@@
 <signal name="YELLOW_LED">
 <contactref element="YELLOW" pad="A"/>
-<contactref element="ESP32" pad="7"/>
-<wire x1="62.23" y1="6.35" x2="58.166" y2="2.286" width="0.508" layer="1"/>
 <wire x1="11.684" y1="18.161" x2="11.684" y2="6.731" width="0.508" layer="1"/>
-<wire x1="58.166" y1="2.286" x2="16.129" y2="2.286" width="0.508" layer="1"/>
+<wire x1="58.166" y1="2.286" x2="57.023" y2="2.286" width="0.508" layer="1"/>
+<wire x1="57.023" y1="2.286" x2="16.129" y2="2.286" width="0.508" layer="1"/>
 <wire x1="16.129" y1="2.286" x2="11.684" y2="6.731" width="0.508" layer="1"/>
 <wire x1="9.525" y1="20.32" x2="11.684" y2="18.161" width="0.508" layer="1"/>
 <wire x1="3.81" y1="20.32" x2="9.525" y2="20.32" width="0.508" layer="1"/>
+<contactref element="ESP32" pad="9"/>
+<wire x1="67.31" y1="6.35" x2="63.246" y2="2.286" width="0.508" layer="1"/>
+<wire x1="63.246" y1="2.286" x2="58.166" y2="2.286" width="0.508" layer="1"/>
 </signal>
 <signal name="FAN_EN">
@@
 <signal name="SERVO">
 <contactref element="SG90" pad="1"/>
-<contactref element="ESP32" pad="5"/>
-<wire x1="34.925" y1="4.445" x2="33.02" y2="6.35" width="0.508" layer="1"/>
-<wire x1="55.245" y1="4.445" x2="34.925" y2="4.445" width="0.508" layer="1"/>
-<wire x1="57.15" y1="6.35" x2="55.245" y2="4.445" width="0.508" layer="1"/>
+<wire x1="35.052" y1="4.318" x2="33.02" y2="6.35" width="0.508" layer="1"/>
+<contactref element="ESP32" pad="7"/>
+<wire x1="60.198" y1="4.318" x2="35.052" y2="4.318" width="0.508" layer="1"/>
+<wire x1="62.23" y1="6.35" x2="60.198" y2="4.318" width="0.508" layer="1"/>
 </signal>
 <signal name="N$5">
@@
 <wire x1="28.448" y1="38.1" x2="28.448" y2="50.927" width="0.508" layer="1"/>
 </signal>
-<signal name="GREEN_LED">
-<contactref element="GREEN" pad="A"/>
-<contactref element="ESP32" pad="6"/>
-<wire x1="59.69" y1="6.35" x2="56.642" y2="3.302" width="0.508" layer="1"/>
-<wire x1="56.642" y1="3.302" x2="19.939" y2="3.302" width="0.508" layer="1"/>
-<wire x1="19.939" y1="3.302" x2="13.97" y2="9.271" width="0.508" layer="1"/>
-<wire x1="13.97" y1="27.432" x2="13.97" y2="9.271" width="0.508" layer="1"/>
-<wire x1="12.192" y1="29.21" x2="13.97" y2="27.432" width="0.508" layer="1"/>
-<wire x1="3.81" y1="29.21" x2="12.192" y2="29.21" width="0.508" layer="1"/>
-</signal>
-<signal name="N$8">
+<signal name="GREEN_R3">
 <contactref element="GREEN" pad="K"/>
 <contactref element="R3" pad="1"/>
 <wire x1="3.81" y1="31.75" x2="10.16" y2="38.1" width="0.508" layer="1"/>
 </signal>
-<signal name="N$21">
+<signal name="RED_R1">
 <contactref element="RED" pad="K"/>
 <contactref element="R1" pad="1"/>
@@
 <wire x1="8.89" y1="13.97" x2="10.16" y2="12.7" width="0.508" layer="1"/>
 </signal>
-<signal name="N$1">
+<signal name="ESP_PWR">
 <contactref element="ESP32" pad="1"/>
-<contactref element="PWR" pad="1"/>
+<contactref element="ESP_PWR" pad="1"/>
 <wire x1="38.1" y1="11.43" x2="43.18" y2="6.35" width="0.762" layer="1"/>
 <wire x1="43.18" y1="6.35" x2="46.99" y2="6.35" width="0.762" layer="1"/>
 </signal>
+<signal name="GREEN_LED">
+<contactref element="GREEN" pad="A"/>
+<contactref element="ESP32" pad="8"/>
+<wire x1="64.77" y1="6.35" x2="61.722" y2="3.302" width="0.508" layer="1"/>
+<wire x1="19.177" y1="3.302" x2="14.224" y2="8.255" width="0.508" layer="1"/>
+<wire x1="14.224" y1="8.255" x2="14.224" y2="26.924" width="0.508" layer="1"/>
+<wire x1="14.224" y1="26.924" x2="11.938" y2="29.21" width="0.508" layer="1"/>
+<wire x1="11.938" y1="29.21" x2="3.81" y2="29.21" width="0.508" layer="1"/>
+<wire x1="61.722" y1="3.302" x2="19.177" y2="3.302" width="0.508" layer="1"/>
+</signal>
+<signal name="RED_LED">
+<contactref element="ESP32" pad="10"/>
+<contactref element="RED" pad="A"/>
+<wire x1="64.77" y1="1.27" x2="69.85" y2="6.35" width="0.508" layer="1"/>
+<wire x1="3.81" y1="11.43" x2="13.97" y2="1.27" width="0.508" layer="1"/>
+<wire x1="13.97" y1="1.27" x2="64.77" y2="1.27" width="0.508" layer="1"/>
+</signal>
 </signals>
