File: schematic.brd (EAGLE design)
At the start: 99.7 x 58.4 mm, 26 parts

Commit message: adefd
Parts:
- INCAP: value 0.2uF -> 470uF
- moved INCAP 6.48 mm to (27.9, 6.35), turned to 0 degrees
Routing:
- net +5V: track 42.1 -> 39.5 mm
- net GREEN_R3: track 8.98 -> 11.2 mm
Changed lines of the file:
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@@
 <attribute name="VALUE" x="14.605" y="52.705" size="1.27" layer="27" rot="R270"/>
 </element>
-<element name="INCAP" library="rcl" library_urn="urn:adsk.eagle:library:334" package="E2,5RE" package3d_urn="urn:adsk.eagle:package:23343/1" value="0.2uF" x="21.59" y="5.08" smashed="yes" rot="R180">
-<attribute name="NAME" x="23.749" y="2.794" size="0.635" layer="25" ratio="10" rot="R180"/>
-<attribute name="SPICEPREFIX" value="C" x="21.59" y="5.08" size="1.778" layer="27" rot="R180" display="off"/>
-<attribute name="VALUE" x="20.955" y="7.366" size="1.27" layer="27" ratio="10" rot="R180"/>
+<element name="INCAP" library="rcl" library_urn="urn:adsk.eagle:library:334" package="E2,5RE" package3d_urn="urn:adsk.eagle:package:23343/1" value="470uF" x="27.94" y="6.35" smashed="yes">
+<attribute name="NAME" x="25.781" y="8.636" size="0.635" layer="25" ratio="10"/>
+<attribute name="SPICEPREFIX" value="C" x="27.94" y="6.35" size="1.778" layer="27" display="off"/>
+<attribute name="VALUE" x="28.575" y="4.064" size="1.27" layer="27" ratio="10"/>
 </element>
 <element name="U$2" library="mine" package="BUCK-CONVERTER" value="BUCK-CONVERTER" x="30.48" y="25.4" smashed="yes" rot="R270"/>
@@
 <contactref element="U$2" pad="VOUT1"/>
 <contactref element="U$2" pad="VOUT2"/>
-<wire x1="22.86" y1="5.08" x2="22.86" y2="6.858" width="1.27" layer="1"/>
-<wire x1="22.86" y1="6.858" x2="26.67" y2="10.668" width="1.27" layer="1"/>
+<wire x1="26.67" y1="6.35" x2="26.67" y2="10.668" width="1.27" layer="1"/>
 <contactref element="SG90" pad="2"/>
 <wire x1="30.48" y1="24.13" x2="27.94" y2="21.59" width="1.27" layer="1"/>
@@
 <wire x1="36.83" y1="24.13" x2="30.48" y2="24.13" width="1.27" layer="1"/>
 <wire x1="35.56" y1="8.382" x2="35.56" y2="6.35" width="1.27" layer="1"/>
-<wire x1="29.21" y1="10.668" x2="32.385" y2="10.668" width="1.27" layer="1"/>
-<wire x1="32.385" y1="10.668" x2="35.56" y2="8.382" width="1.27" layer="1"/>
 <wire x1="29.21" y1="10.668" x2="26.67" y2="10.668" width="1.27" layer="1"/>
 <wire x1="29.21" y1="10.668" x2="27.94" y2="12.192" width="1.27" layer="1"/>
 <wire x1="27.94" y1="12.192" x2="26.67" y2="10.668" width="1.27" layer="1"/>
+<wire x1="29.21" y1="10.668" x2="30.734" y2="9.144" width="1.27" layer="1"/>
+<wire x1="34.798" y1="9.144" x2="35.56" y2="8.382" width="1.27" layer="1"/>
+<wire x1="30.734" y1="9.144" x2="34.798" y2="9.144" width="1.27" layer="1"/>
 </signal>
 <signal name="FAN_PW">
@@
 <contactref element="GREEN" pad="K"/>
 <contactref element="R3" pad="1"/>
-<wire x1="3.81" y1="31.75" x2="10.16" y2="38.1" width="0.508" layer="1"/>
+<wire x1="10.16" y1="38.1" x2="6.35" y2="38.1" width="0.508" layer="1"/>
+<wire x1="6.35" y1="38.1" x2="3.81" y2="35.56" width="0.508" layer="1"/>
+<wire x1="3.81" y1="35.56" x2="3.81" y2="31.75" width="0.508" layer="1"/>
 </signal>
 <signal name="RED_R1">
