File: schematic.sch (EAGLE design)
At the start: 25 parts

Commit message: akjdf;sjf
Parts:
- removed U$1: BUCK-CONVERTER, buck-converter:BUCK-CONVERTER
- added PWR: (no value), pinhead:PINHD-1X2
- added U$2: BUCK-CONVERTER, mine:BUCK-CONVERTER
Connections:
- net MS1_X renamed N$11
- net MS1_Y renamed N$5
- net MS2_X renamed N$12
- net MS2_Y renamed N$9
- net MS3_X renamed N$13
- net MS3_Y renamed N$10
- net N$32 renamed FAN_PW
- removed net N$15: DRIVER_X./EN, ESP32.IO27
- removed net N$19: DRIVER_Y./EN, ESP32.IO33
- removed net N$2: DRIVER_X.STEP, ESP32.IO14
- removed net N$23: ESP32.IO23, RED.A
- removed net N$25: GREEN.C, R1.1
- removed net N$26: ESP32.IO21, GREEN.A
- removed net N$27: ESP32.IO22, YELLOW.A
- removed net N$29: R3.1, RED.C
- removed net N$30: ESP32.IO32, SG90.SIG
- removed net N$31: ESP32.IO17, IRL540N.G, R4.1
- removed net N$4: DRIVER_Y.DIR, ESP32.IO26
- removed net N$5 (its old number): DRIVER_Y.STEP, ESP32.IO25
- new net FAN_EN: ESP32.IO0, IRL540N.G, R4.1
- new net GREEN_LED: ESP32.IO35, GREEN.A
- new net N$21: R1.1, RED.C
- new net N$8: GREEN.C, R3.1
- new net RED_LED: ESP32.IO33, RED.A
- new net SERVO: ESP32.IO34, SG90.SIG
- new net X_DIR: DRIVER_X.DIR, ESP32.IO19
- new net X_EN: DRIVER_X./EN, ESP32.IO5
- new net X_STEP: DRIVER_X.STEP, ESP32.IO18
- new net YELLOW_LED: ESP32.IO32, YELLOW.A
- new net Y_DIR: DRIVER_Y.DIR, ESP32.IO21
- new net Y_EN: DRIVER_Y./EN, ESP32.IO23
- new net Y_STEP: DRIVER_Y.STEP, ESP32.IO22
- net +12V: now also U$2.VIN; no longer U$1.VIN
- net +3V3: now also PWR.2; no longer ESP32.3V3
- net +5V: now also U$2.VOUT; no longer U$1.VOUT
- net GND: now also U$2.GND@1, U$2.GND@2; no longer U$1.GND@1, U$1.GND@2
- net N$1: now also ESP32.3V3, PWR.1; no longer DRIVER_X.DIR, ESP32.IO12
Other:
- moved on the sheet: DRIVER_X, DRIVER_Y, ESP32, FAN1, FAN2, GREEN, INCAP, IRL540N, LF33CV, MICROSTEP_X, MICROSTEP_Y, MOTOR_X-1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

Commit message: kasjf;lkdsjf
Parts:
- renumbered PWR to ESP_PWR
Connections:
- net N$1 renamed ESP_PWR
- net N$21 renamed RED_R1
- net N$7 renamed YELLOW_R2
- net N$8 renamed GREEN_R3
- net GREEN_LED: now also ESP32.IO33; no longer ESP32.IO35
- net RED_LED: now also ESP32.IO26; no longer ESP32.IO33
- net SERVO: now also ESP32.IO32; no longer ESP32.IO34
- net YELLOW_LED: now also ESP32.IO25; no longer ESP32.IO32
Other:
- moved on the sheet: GREEN, R1, R2, R3, RED, YELLOW
Changed lines of the file:
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@@
 <part name="GND10" library="supply1" library_urn="urn:adsk.eagle:library:371" deviceset="GND" device=""/>
 <part name="U$2" library="mine" deviceset="BUCK-CONVERTER" device=""/>
-<part name="PWR" library="pinhead" library_urn="urn:adsk.eagle:library:325" deviceset="PINHD-1X2" device="" package3d_urn="urn:adsk.eagle:package:22435/2"/>
+<part name="ESP_PWR" library="pinhead" library_urn="urn:adsk.eagle:library:325" deviceset="PINHD-1X2" device="" package3d_urn="urn:adsk.eagle:package:22435/2"/>
 </parts>
 <sheets>
@@
 <attribute name="NAME" x="147.32" y="51.435" size="1.778" layer="95"/>
 </instance>
-<instance part="GREEN" gate="G$1" x="50.8" y="38.1" smashed="yes">
-<attribute name="NAME" x="54.356" y="33.528" size="1.778" layer="95" rot="R90"/>
-<attribute name="VALUE" x="56.515" y="33.528" size="1.778" layer="96" rot="R90"/>
-</instance>
-<instance part="YELLOW" gate="G$1" x="60.96" y="38.1" smashed="yes">
-<attribute name="NAME" x="64.516" y="33.528" size="1.778" layer="95" rot="R90"/>
-<attribute name="VALUE" x="66.675" y="33.528" size="1.778" layer="96" rot="R90"/>
-</instance>
-<instance part="RED" gate="G$1" x="71.12" y="38.1" smashed="yes">
-<attribute name="NAME" x="74.676" y="33.528" size="1.778" layer="95" rot="R90"/>
-<attribute name="VALUE" x="76.835" y="33.528" size="1.778" layer="96" rot="R90"/>
-</instance>
-<instance part="R1" gate="G$1" x="71.12" y="25.4" smashed="yes" rot="R270">
-<attribute name="NAME" x="72.6186" y="29.21" size="1.778" layer="95" rot="R270"/>
-<attribute name="VALUE" x="67.818" y="29.21" size="1.778" layer="96" rot="R270"/>
-</instance>
-<instance part="R2" gate="G$1" x="60.96" y="25.4" smashed="yes" rot="R270">
-<attribute name="NAME" x="62.4586" y="29.21" size="1.778" layer="95" rot="R270"/>
-<attribute name="VALUE" x="57.658" y="29.21" size="1.778" layer="96" rot="R270"/>
-</instance>
-<instance part="R3" gate="G$1" x="50.8" y="25.4" smashed="yes" rot="R270">
-<attribute name="NAME" x="52.2986" y="29.21" size="1.778" layer="95" rot="R270"/>
-<attribute name="VALUE" x="47.498" y="29.21" size="1.778" layer="96" rot="R270"/>
+<instance part="GREEN" gate="G$1" x="55.88" y="38.1" smashed="yes">
+<attribute name="NAME" x="59.436" y="33.528" size="1.778" layer="95" rot="R90"/>
+<attribute name="VALUE" x="61.595" y="33.528" size="1.778" layer="96" rot="R90"/>
+</instance>
+<instance part="YELLOW" gate="G$1" x="66.04" y="38.1" smashed="yes">
+<attribute name="NAME" x="69.596" y="33.528" size="1.778" layer="95" rot="R90"/>
+<attribute name="VALUE" x="71.755" y="33.528" size="1.778" layer="96" rot="R90"/>
+</instance>
+<instance part="RED" gate="G$1" x="76.2" y="38.1" smashed="yes">
+<attribute name="NAME" x="79.756" y="33.528" size="1.778" layer="95" rot="R90"/>
+<attribute name="VALUE" x="81.915" y="33.528" size="1.778" layer="96" rot="R90"/>
+</instance>
+<instance part="R1" gate="G$1" x="76.2" y="25.4" smashed="yes" rot="R270">
+<attribute name="NAME" x="77.6986" y="29.21" size="1.778" layer="95" rot="R270"/>
+<attribute name="VALUE" x="72.898" y="29.21" size="1.778" layer="96" rot="R270"/>
+</instance>
+<instance part="R2" gate="G$1" x="66.04" y="25.4" smashed="yes" rot="R270">
+<attribute name="NAME" x="67.5386" y="29.21" size="1.778" layer="95" rot="R270"/>
+<attribute name="VALUE" x="62.738" y="29.21" size="1.778" layer="96" rot="R270"/>
+</instance>
+<instance part="R3" gate="G$1" x="55.88" y="25.4" smashed="yes" rot="R270">
+<attribute name="NAME" x="57.3786" y="29.21" size="1.778" layer="95" rot="R270"/>
+<attribute name="VALUE" x="52.578" y="29.21" size="1.778" layer="96" rot="R270"/>
 </instance>
 <instance part="R4" gate="G$1" x="99.06" y="68.58" smashed="yes" rot="R270">
@@
 <attribute name="VALUE" x="134.62" y="50.8" size="1.778" layer="96" rot="R90"/>
 </instance>
-<instance part="GND5" gate="1" x="60.96" y="10.16" smashed="yes">
-<attribute name="VALUE" x="58.42" y="7.62" size="1.778" layer="96"/>
+<instance part="GND5" gate="1" x="66.04" y="10.16" smashed="yes">
+<attribute name="VALUE" x="63.5" y="7.62" size="1.778" layer="96"/>
 </instance>
 <instance part="GND6" gate="1" x="15.24" y="53.34" smashed="yes" rot="R180">
@@
 </instance>
 <instance part="U$2" gate="G$1" x="106.68" y="40.64" smashed="yes"/>
-<instance part="PWR" gate="G$1" x="43.18" y="43.18" smashed="yes">
+<instance part="ESP_PWR" gate="G$1" x="43.18" y="43.18" smashed="yes">
 <attribute name="NAME" x="36.83" y="48.895" size="1.778" layer="95"/>
 <attribute name="VALUE" x="36.83" y="38.1" size="1.778" layer="96"/>
@@
 </segment>
 <segment>
-<wire x1="71.12" y1="17.78" x2="60.96" y2="17.78" width="0.1524" layer="91"/>
-<wire x1="60.96" y1="17.78" x2="50.8" y2="17.78" width="0.1524" layer="91"/>
+<wire x1="76.2" y1="17.78" x2="66.04" y2="17.78" width="0.1524" layer="91"/>
+<wire x1="66.04" y1="17.78" x2="55.88" y2="17.78" width="0.1524" layer="91"/>
 <pinref part="R2" gate="G$1" pin="2"/>
-<wire x1="60.96" y1="20.32" x2="60.96" y2="17.78" width="0.1524" layer="91"/>
-<junction x="60.96" y="17.78"/>
+<wire x1="66.04" y1="20.32" x2="66.04" y2="17.78" width="0.1524" layer="91"/>
+<junction x="66.04" y="17.78"/>
 <pinref part="GND5" gate="1" pin="GND"/>
-<wire x1="60.96" y1="17.78" x2="60.96" y2="12.7" width="0.1524" layer="91"/>
+<wire x1="66.04" y1="17.78" x2="66.04" y2="12.7" width="0.1524" layer="91"/>
 <pinref part="R1" gate="G$1" pin="2"/>
-<wire x1="71.12" y1="20.32" x2="71.12" y2="17.78" width="0.1524" layer="91"/>
+<wire x1="76.2" y1="20.32" x2="76.2" y2="17.78" width="0.1524" layer="91"/>
 <pinref part="R3" gate="G$1" pin="2"/>
-<wire x1="50.8" y1="20.32" x2="50.8" y2="17.78" width="0.1524" layer="91"/>
+<wire x1="55.88" y1="20.32" x2="55.88" y2="17.78" width="0.1524" layer="91"/>
 </segment>
 <segment>
@@
 </segment>
 <segment>
-<pinref part="PWR" gate="G$1" pin="2"/>
+<pinref part="ESP_PWR" gate="G$1" pin="2"/>
 <wire x1="40.64" y1="43.18" x2="38.1" y2="43.18" width="0.1524" layer="91"/>
 <pinref part="+3V2" gate="G$1" pin="+3V3"/>
@@
 </segment>
 </net>
-<net name="RED_LED" class="0">
-<segment>
-<pinref part="ESP32" gate="G$1" pin="IO33"/>
-<wire x1="55.88" y1="58.42" x2="55.88" y2="48.26" width="0.1524" layer="91"/>
-<wire x1="55.88" y1="48.26" x2="71.12" y2="48.26" width="0.1524" layer="91"/>
-<pinref part="RED" gate="G$1" pin="A"/>
-<wire x1="71.12" y1="48.26" x2="71.12" y2="40.64" width="0.1524" layer="91"/>
-</segment>
-</net>
 <net name="FAN_PW" class="0">
 <segment>
@@
 </segment>
 </net>
-<net name="N$7" class="0">
+<net name="YELLOW_R2" class="0">
 <segment>
 <pinref part="R2" gate="G$1" pin="1"/>
 <pinref part="YELLOW" gate="G$1" pin="C"/>
-<wire x1="60.96" y1="30.48" x2="60.96" y2="33.02" width="0.1524" layer="91"/>
+<wire x1="66.04" y1="30.48" x2="66.04" y2="33.02" width="0.1524" layer="91"/>
 </segment>
 </net>
@@
 <segment>
 <pinref part="YELLOW" gate="G$1" pin="A"/>
-<wire x1="60.96" y1="40.64" x2="60.96" y2="45.72" width="0.1524" layer="91"/>
-<pinref part="ESP32" gate="G$1" pin="IO32"/>
-<wire x1="53.34" y1="58.42" x2="53.34" y2="45.72" width="0.1524" layer="91"/>
-<wire x1="53.34" y1="45.72" x2="60.96" y2="45.72" width="0.1524" layer="91"/>
+<wire x1="66.04" y1="40.64" x2="66.04" y2="45.72" width="0.1524" layer="91"/>
+<pinref part="ESP32" gate="G$1" pin="IO25"/>
+<wire x1="58.42" y1="58.42" x2="58.42" y2="45.72" width="0.1524" layer="91"/>
+<wire x1="58.42" y1="45.72" x2="66.04" y2="45.72" width="0.1524" layer="91"/>
 </segment>
 </net>
@@
 <pinref part="SG90" gate="G$1" pin="SIG"/>
 <wire x1="20.32" y1="45.72" x2="20.32" y2="50.8" width="0.1524" layer="91"/>
-<wire x1="20.32" y1="50.8" x2="48.26" y2="50.8" width="0.1524" layer="91"/>
-<pinref part="ESP32" gate="G$1" pin="IO34"/>
-<wire x1="48.26" y1="50.8" x2="48.26" y2="58.42" width="0.1524" layer="91"/>
+<wire x1="20.32" y1="50.8" x2="53.34" y2="50.8" width="0.1524" layer="91"/>
+<pinref part="ESP32" gate="G$1" pin="IO32"/>
+<wire x1="53.34" y1="50.8" x2="53.34" y2="58.42" width="0.1524" layer="91"/>
 </segment>
 </net>
@@
 </segment>
 </net>
-<net name="GREEN_LED" class="0">
-<segment>
-<pinref part="GREEN" gate="G$1" pin="A"/>
-<pinref part="ESP32" gate="G$1" pin="IO35"/>
-<wire x1="50.8" y1="40.64" x2="50.8" y2="58.42" width="0.1524" layer="91"/>
-</segment>
-</net>
-<net name="N$8" class="0">
+<net name="GREEN_R3" class="0">
 <segment>
 <pinref part="GREEN" gate="G$1" pin="C"/>
 <pinref part="R3" gate="G$1" pin="1"/>
-<wire x1="50.8" y1="33.02" x2="50.8" y2="30.48" width="0.1524" layer="91"/>
-</segment>
-</net>
-<net name="N$21" class="0">
+<wire x1="55.88" y1="33.02" x2="55.88" y2="30.48" width="0.1524" layer="91"/>
+</segment>
+</net>
+<net name="RED_R1" class="0">
 <segment>
 <pinref part="RED" gate="G$1" pin="C"/>
 <pinref part="R1" gate="G$1" pin="1"/>
-<wire x1="71.12" y1="33.02" x2="71.12" y2="30.48" width="0.1524" layer="91"/>
-</segment>
-</net>
-<net name="N$1" class="0">
+<wire x1="76.2" y1="33.02" x2="76.2" y2="30.48" width="0.1524" layer="91"/>
+</segment>
+</net>
+<net name="ESP_PWR" class="0">
 <segment>
 <pinref part="ESP32" gate="G$1" pin="3V3"/>
 <wire x1="38.1" y1="58.42" x2="38.1" y2="45.72" width="0.1524" layer="91"/>
-<pinref part="PWR" gate="G$1" pin="1"/>
+<pinref part="ESP_PWR" gate="G$1" pin="1"/>
 <wire x1="38.1" y1="45.72" x2="40.64" y2="45.72" width="0.1524" layer="91"/>
 </segment>
 </net>
+<net name="GREEN_LED" class="0">
+<segment>
+<pinref part="GREEN" gate="G$1" pin="A"/>
+<pinref part="ESP32" gate="G$1" pin="IO33"/>
+<wire x1="55.88" y1="40.64" x2="55.88" y2="58.42" width="0.1524" layer="91"/>
+</segment>
+</net>
+<net name="RED_LED" class="0">
+<segment>
+<pinref part="ESP32" gate="G$1" pin="IO26"/>
+<wire x1="60.96" y1="58.42" x2="60.96" y2="48.26" width="0.1524" layer="91"/>
+<wire x1="60.96" y1="48.26" x2="76.2" y2="48.26" width="0.1524" layer="91"/>
+<pinref part="RED" gate="G$1" pin="A"/>
+<wire x1="76.2" y1="48.26" x2="76.2" y2="40.64" width="0.1524" layer="91"/>
+</segment>
+</net>

Commit message: adefd
Parts:
- INCAP: value 0.2uF -> 470uF
Changed lines of the file:
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@@
 <part name="GND7" library="supply1" library_urn="urn:adsk.eagle:library:371" deviceset="GND" device=""/>
 <part name="P+6" library="supply1" library_urn="urn:adsk.eagle:library:371" deviceset="+12V" device=""/>
-<part name="INCAP" library="rcl" library_urn="urn:adsk.eagle:library:334" deviceset="CPOL-EU" device="E2.5-4V" package3d_urn="urn:adsk.eagle:package:23343/1" value="0.2uF"/>
+<part name="INCAP" library="rcl" library_urn="urn:adsk.eagle:library:334" deviceset="CPOL-EU" device="E2.5-4V" package3d_urn="urn:adsk.eagle:package:23343/1" value="470uF"/>
 <part name="GND8" library="supply1" library_urn="urn:adsk.eagle:library:371" deviceset="GND" device=""/>
 <part name="GND9" library="supply1" library_urn="urn:adsk.eagle:library:371" deviceset="GND" device=""/>
